File: airMouse-pcb/mouse.kicad_sch (KiCad schematic)
At the start: 40 parts, among them SW50 KEY, SW51 KEY, SW52 KEY, SW53 KEY, SW54 KEY, SW55 KEY, SW56 KEY, SW57 KEY, SW58 KEY, SW59 KEY

Commit message: page data
Other:
- company: (none) -> Bart's Design
- title: (none) -> EtherPointer
Changed lines of the file:
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@@
 	(generator_version "8.0")
 	(paper "A4")
+	(title_block
+		(title "EtherPointer")
+		(date "2025-02-13")
+		(rev "RC1")
+		(company "Bart's Design")
+		(comment 1 "Bartosz Pracz")
+	)
 	(junction
 		(at 31.75 77.47)
