File: hardware/airMouse-mouse/airMouse-mouse.kicad_pcb (KiCad board)
At the start: 2 copper layers, 85.2 x 42 mm, 222 parts, among them J4 AT, J5 RADIO_PRG, J6 MCU_PRG, Q1 IRLML6346, SW1 KEY, SW10 KEY, SW11 KEY, SW12 KEY, SW13 KEY, SW14 KEY, SW15 KEY, SW16 KEY, SW17 KEY, SW18 KEY, SW19 KEY, SW2 KEY, SW20 KEY, SW21 KEY, SW22 KEY, SW23 KEY, SW24 KEY, SW25 KEY, SW26 KEY, SW27 KEY, SW28 KEY, SW29 KEY, SW3 KEY, SW30 KEY, SW31 KEY, SW32 KEY, SW33 KEY, SW34 KEY, SW35 KEY, SW36 KEY, SW37 KEY, SW38 KEY, SW39 KEY, SW4 KEY, SW40 KEY, SW41 KEY, SW42 KEY, SW43 KEY, SW44 KEY, SW45 KEY, SW46 KEY, SW47 KEY, SW48 KEY, SW49 KEY, SW5 KEY, SW50 KEY, SW51 KEY, SW52 KEY, SW53 KEY, SW54 KEY, SW55 KEY, SW56 KEY, SW57 KEY, SW58 KEY, SW59 KEY, SW6 KEY, SW60 KEY, SW7 KEY, SW8 KEY, SW9 KEY, U1 STM32G071RBTx, U2 AP1603, U3 ESP32-C3-WROOM-02U, U4 LSM6DS3

Commit message: add mouse pcb
Parts:
- removed BT1: BC-0401, airMouseLib:BC-0401
- removed C1: 105, Capacitor_SMD:C_0603_1608Metric
- removed C10, C11, C12, C13, C14, C15, C16, C17, C18, C19, C2, C20, C21, C22, C23, C24, C25, C26, C29, C31, C33, C34, C5, C6, C7, C8, C9: 100n, Capacitor_SMD:C_0603_1608Metric
- removed C27: 4u7, Capacitor_SMD:C_0805_2012Metric
- removed C28, C30: 1u, Capacitor_SMD:C_0603_1608Metric
- removed C3, C4: 47u, Capacitor_SMD:CP_Elec_6.3x5.8
- removed C32: 10u, Capacitor_SMD:C_0805_2012Metric
- removed D1: MBR0530, Diode_SMD:D_SOD-123
- removed D10, D11, D14, D15, D16, D17, D18, D19, D2, D20, D21, D22, D23, D24, D25, D26, D27, D28, D29, D3, D30, D31, D32, D33, D34, D35, D36, D37, D38, D39, D4, D40, D41, D42, D44, D45, D46, D47, D5, D50, D51, D54, D55, D58, D59, D6, D7, D8, D9: BAS70X-TP, Diode_SMD:D_SOD-523
- removed D12: STBY, LED_SMD:LED_0603_1608Metric
- removed D13: BT, LED_SMD:LED_0603_1608Metric
- removed D43: LOW_BAT, LED_SMD:LED_0603_1608Metric
- removed FB1: 600R @ 100M, Capacitor_SMD:C_0603_1608Metric
- removed J4: AT, Connector_JST:JST_ZH_S3B-ZR-SM4A-TF_1x03-1MP_P1.50mm_Horizontal
- removed J5: RADIO_PRG, Connector_JST:JST_ZH_S3B-ZR-SM4A-TF_1x03-1MP_P1.50mm_Horizontal
- removed J6: MCU_PRG, Connector_JST:JST_ZH_S5B-ZR-SM4A-TF_1x05-1MP_P1.50mm_Horizontal
- removed L1: 22u / WLPN303010M220PB, Inductor_SMD:L_Abracon_ASPI-3012S
- removed LD1: 70115420, Connector_PinHeader_2.54mm:PinHeader_1x02_P2.54mm_Vertical
- removed Q1: IRLML6346, Package_TO_SOT_SMD:SOT-23
- removed R10, R11, R12, R16, R17, R18, R19, R20, R21, R22, R23, R24, R25, R26, R27, R28, R29, R30, R31, R32, R33, R34, R35, R36, R37, R38, R39, R40, R41, R42, R43, R44, R45, R49, R50, R53, R54, R55, R56, R58, R59, R9: 10k, Resistor_SMD:R_0603_1608Metric
- removed R13, R14, R15: 100R, Resistor_SMD:R_0603_1608Metric
- removed R46, R47, R48, R57: 2k2, Resistor_SMD:R_0603_1608Metric
- removed R51, R52: 4k7, Resistor_SMD:R_0603_1608Metric
- removed R60, R61: 0R, Resistor_SMD:R_0603_1608Metric
- removed SW10, SW11, SW12, SW13, SW14, SW15, SW16, SW17, SW18, SW19, SW20, SW21, SW22, SW23, SW24, SW25, SW26, SW27, SW28, SW29, SW30, SW31, SW32, SW33, SW34, SW35, SW36, SW37, SW38, SW39, SW40, SW41, SW42, SW43, SW44, SW45, SW46, SW47, SW48, SW49, SW50, SW51, SW52, SW53, SW54, SW55, SW56, SW57, SW58, SW59, SW60, SW9: KEY, airMouseLib:TL3315NF100Q
- removed TP1: DBG_TX, TestPoint:TestPoint_Pad_D1.0mm
- removed TP2: DBG_RX, TestPoint:TestPoint_Pad_D1.0mm
- removed U1: STM32G071RBTx, Package_QFP:LQFP-64_10x10mm_P0.5mm
- removed U2: AP1603, Package_TO_SOT_SMD:SOT-23-6
- removed U3: ESP32-C3-WROOM-02U, RF_Module:ESP32-C3-WROOM-02U
- removed U4: LSM6DS3, Package_LGA:LGA-14_3x2.5mm_P0.5mm_LayoutBorder3x4y
- added J1: DS1020-07-10VBT1A-R, airMouseLib:DS1020-07-10VBT1A-R, F.Cu at (159.2, 80.0)
- added Logo1: ~, airMouseLib:Bart's Design 30mm, B.Cu at (135.0, 80.0)
- R1, R2: value 100R -> 10k
- moved SW3 49.0 mm to (147.0, 73.0)
- moved R8 46.1 mm to (156.5, 73.2), turned to -90 degrees
- moved SW2 39.6 mm to (133.5, 80.0)
- moved SW1 34.0 mm to (120.0, 73.0)
- moved SW4 31.3 mm to (133.5, 73.0)
- moved SW6 30.5 mm to (147.0, 87.0)
- moved SW5 22.5 mm to (133.5, 87.0)
- moved R7 22.3 mm to (155.0, 73.2), turned to -90 degrees
- moved R6 19.8 mm to (153.5, 73.2), turned to -90 degrees
- moved SW7 18.0 mm to (140.0, 87.0)
- moved R5 17.4 mm to (152.0, 73.2), turned to -90 degrees
- moved R2 15.6 mm to (155.0, 87.0), turned to 90 degrees
- moved R1 15.5 mm to (156.5, 87.0), turned to 90 degrees
- moved R3 9.99 mm to (153.5, 87.0), turned to 90 degrees
- moved R4 8.19 mm to (152.0, 87.0), turned to 90 degrees
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Connections:
- R1 pad 1: /Keyboard/KEY_ROW1 -> +3V3
- R1 pad 2: Net-(D10-K) -> /LMB
- R2 pad 1: /Keyboard/KEY_ROW2 -> +3V3
- R2 pad 2: Net-(D14-K) -> /MMB
- R3 pad 2: Net-(SW1-A) -> /RMB
- R4 pad 2: Net-(SW12-A) -> /SCRLUP
- R5 pad 2: Net-(SW13-A) -> /SCRLDN
- R6 pad 2: Net-(SW14-A) -> /DPI
- R7 pad 2: Net-(SW15-A) -> /PRECISION
- R8 pad 2: Net-(SW16-A) -> /HOME
- SW1 pad 1: Net-(SW1-A) -> GND
- SW1 pad 2: Net-(D2-A) -> /LMB
- SW2 pad 1: Net-(SW12-A) -> GND
- SW2 pad 2: Net-(D3-A) -> /MMB
- SW3 pad 1: Net-(SW13-A) -> GND
- SW3 pad 2: Net-(D4-A) -> /RMB
- SW4 pad 1: Net-(SW14-A) -> GND
- SW4 pad 2: Net-(D5-A) -> /SCRLUP
- SW5 pad 1: Net-(SW15-A) -> GND
- SW5 pad 2: Net-(D6-A) -> /SCRLDN
- SW6 pad 1: Net-(SW16-A) -> GND
- SW6 pad 2: Net-(D7-A) -> /DPI
- SW7 pad 1: Net-(SW17-A) -> GND
- SW7 pad 2: Net-(D8-A) -> /PRECISION
- SW8 pad 1: Net-(SW18-A) -> GND
- SW8 pad 2: Net-(D9-A) -> /HOME
Routing:
- net Net-(SW1-A): track 94.2 -> 0.00 mm, vias 4 -> 0
- net Net-(SW12-A): track 89.9 -> 0.00 mm, vias 4 -> 0
- net Net-(SW13-A): track 88.7 -> 0.00 mm, vias 4 -> 0
- net Net-(SW14-A): track 87.6 -> 0.00 mm, vias 4 -> 0
- net Net-(SW15-A): track 85.2 -> 0.00 mm, vias 4 -> 0
- net Net-(D14-K): track 68.7 -> 0.00 mm, vias 1 -> 0
- net Net-(SW16-A): track 68.5 -> 0.00 mm, vias 2 -> 0
- net Net-(D22-K): track 64.7 -> 0.00 mm, vias 3 -> 0
- net Net-(D10-K): track 64.6 -> 0.00 mm, vias 1 -> 0
- net Net-(D26-K): track 64.3 -> 0.00 mm, vias 1 -> 0
- net Net-(D18-K): track 63.0 -> 0.00 mm, vias 1 -> 0
- net Net-(SW17-A): track 62.3 -> 0.00 mm, vias 2 -> 0
- net Net-(SW18-A): track 57.6 -> 0.00 mm, vias 4 -> 0
- net /LMB: track 0.00 -> 54.5 mm, vias 0 -> 2
- net /HOME: track 0.00 -> 54.0 mm, vias 0 -> 2
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- added copper zone on B.Cu, net GND
- added copper zone on F.Cu, net GND
Other:
- board size 85.2 x 42 mm -> 50 x 23 mm
- board text added: "airMouse-mouse RC1"
