File: hardware/airMouse-mouse/airMouse-mouse.kicad_sch (KiCad schematic)
At the start: 51 parts, among them J4 AT, J5 RADIO_PRG, J6 MCU_PRG, Q1 IRLML6346, SW60 KEY, U1 STM32G071RBTx, U2 AP1603, U3 ESP32-C3-WROOM-02U, U4 LSM6DS3

Commit message: add mouse pcb
Parts:
- removed BT1: BC-0401, airMouseLib:BC-0401, symbol Device:Battery_Cell
- removed C1: 105, Capacitor_SMD:C_0603_1608Metric, symbol Device:C
- removed C2, C26, C29, C31, C33, C34, C35, C5: 100n, Capacitor_SMD:C_0603_1608Metric, symbol Device:C
- removed C27: 4u7, Capacitor_SMD:C_0805_2012Metric, symbol Device:C
- removed C28, C30: 1u, Capacitor_SMD:C_0603_1608Metric, symbol Device:C
- removed C3, C4: 47u, Capacitor_SMD:CP_Elec_6.3x5.8, symbol Device:C_Polarized
- removed C32: 10u, Capacitor_SMD:C_0805_2012Metric, symbol Device:C
- removed D1: MBR0530, Diode_SMD:D_SOD-123, symbol Device:D_Schottky
- removed D12: STBY, LED_SMD:LED_0603_1608Metric, symbol Device:LED
- removed D13: BT, LED_SMD:LED_0603_1608Metric, symbol Device:LED
- removed D43: LOW_BAT, LED_SMD:LED_0603_1608Metric, symbol Device:LED
- removed FB1: 600R @ 100M, Capacitor_SMD:C_0603_1608Metric, symbol Device:FerriteBead
- removed J4: AT, Connector_JST:JST_ZH_S3B-ZR-SM4A-TF_1x03-1MP_P1.50mm_Horizontal, symbol airMouseLib:Conn_01x03_MP
- removed J5: RADIO_PRG, Connector_JST:JST_ZH_S3B-ZR-SM4A-TF_1x03-1MP_P1.50mm_Horizontal, symbol airMouseLib:Conn_01x03_MP
- removed J6: MCU_PRG, Connector_JST:JST_ZH_S5B-ZR-SM4A-TF_1x05-1MP_P1.50mm_Horizontal, symbol airMouseLib:Conn_01x05_MP
- removed L1: 22u / WLPN303010M220PB, Inductor_SMD:L_Abracon_ASPI-3012S, symbol Device:L
- removed LD1: 70115420, Connector_PinHeader_2.54mm:PinHeader_1x02_P2.54mm_Vertical, symbol Device:D_Laser_1C2A
- removed Q1: IRLML6346, Package_TO_SOT_SMD:SOT-23, symbol Device:Q_NMOS_GSD
- removed R46, R47, R48, R57: 2k2, Resistor_SMD:R_0603_1608Metric, symbol Device:R
- removed R49, R50, R53, R54, R55, R56, R58, R59: 10k, Resistor_SMD:R_0603_1608Metric, symbol Device:R
- removed R51, R52: 4k7, Resistor_SMD:R_0603_1608Metric, symbol Device:R
- removed R60, R61: 0R, Resistor_SMD:R_0603_1608Metric, symbol Device:R
- removed R62: 1k, symbol Device:R
- removed SW60: KEY, airMouseLib:TL3315NF100Q, symbol airMouseLib:KEY
- removed TP1: DBG_TX, TestPoint:TestPoint_Pad_D1.0mm, symbol Connector:TestPoint
- removed TP2: DBG_RX, TestPoint:TestPoint_Pad_D1.0mm, symbol Connector:TestPoint
- removed U1: STM32G071RBTx, Package_QFP:LQFP-64_10x10mm_P0.5mm, symbol MCU_ST_STM32G0:STM32G071RBTx
- removed U2: AP1603, Package_TO_SOT_SMD:SOT-23-6, symbol airMouseLib:AP1603
- removed U3: ESP32-C3-WROOM-02U, RF_Module:ESP32-C3-WROOM-02U, symbol RF_Module:ESP32-C3-WROOM-02U
- removed U4: LSM6DS3, Package_LGA:LGA-14_3x2.5mm_P0.5mm_LayoutBorder3x4y, symbol Sensor_Motion:LSM6DS3
- added J1: DS1020-07-10VBT1A-R, airMouseLib:DS1020-07-10VBT1A-R, symbol Connector_Generic_MountingPin:Conn_01x10_MountingPin
- added Logo1: ~, airMouseLib:Bart's Design 30mm, symbol airMouseLib:Bart's_Design_logo
- added R1, R2, R3, R4, R5, R6, R7, R8: 10k, Resistor_SMD:R_0603_1608Metric, symbol Device:R
- added SW1, SW2, SW3, SW4, SW5, SW6, SW7, SW8: KEY, airMouseLib:TL3315NF100Q, symbol airMouseLib:KEY
Connections:
- net +3V3: now also J1.1 (Pin_1), R1.1, R2.1, R3.1, R4.1, R5.1, R6.1, R7.1, R8.1
- net GND: now also J1.10 (Pin_10), J1.MP (MountPin), SW1.1 (A), SW2.1 (A), SW3.1 (A), SW4.1 (A), SW5.1 (A), SW6.1 (A), SW7.1 (A), SW8.1 (A)
- new net DPI: J1.7 (Pin_7), R6.2, SW6.2 (B)
- new net HOME: J1.9 (Pin_9), R8.2, SW8.2 (B)
- new net LMB: J1.2 (Pin_2), R1.2, SW1.2 (B)
- new net MMB: J1.3 (Pin_3), R2.2, SW2.2 (B)
- new net PRECISION: J1.8 (Pin_8), R7.2, SW7.2 (B)
- new net RMB: J1.4 (Pin_4), R3.2, SW3.2 (B)
- new net SCRLDN: J1.6 (Pin_6), R5.2, SW5.2 (B)
- new net SCRLUP: J1.5 (Pin_5), R4.2, SW4.2 (B)
- no-connect marks 28 -> 0
Other:
- removed sheet Keyboard
- removed sheet mouse
- note added: "keys: TL3315NF100Q"
- note removed: "additional parts: 1x ZH plug ZHR-3 1x ZH plug ZHR-5 8x ZH pin w/ cable SZH-200BK26"
- title: EtherPointer -> EtherPointer mouse
