File: hardware/airMouse-thumb/airMouse-thumb.kicad_pcb (KiCad board)
At the start: 2 copper layers, 21 parts, among them J1 DS1020-07-12VBT1A-R, SW1 KEY, SW10 KEY, SW2 KEY, SW3 KEY, SW4 KEY, SW5 KEY, SW6 KEY, SW7 KEY, SW8 KEY, SW9 KEY

Commit message: thumb pcb
Parts:
- removed R10, R3, R4, R5, R6, R7, R8, R9: 10k, Resistor_SMD:R_0603_1608Metric
- removed SW10, SW3, SW4, SW5, SW6, SW7, SW8, SW9: KEY, airMouseLib:TL3315NF100Q
- added Logo1: ~, airMouseLib:Bart's Design 30mm, B.Cu at (163.8, 60.4)
- J1: value DS1020-07-12VBT1A-R -> DS1020-07-4VBT1A-R; footprint airMouseLib:DS1020-07-12VBT1A-R -> airMouseLib:DS1020-07-4VBT1A-R
- moved R2 64.5 mm to (156.0, 56.0), turned to -90 degrees
- moved J1 62.7 mm to (153.3, 60.0), turned to -90 degrees
- moved SW1 61.4 mm to (178.0, 60.0)
- moved R1 54.8 mm to (156.0, 64.0), turned to 90 degrees
- moved SW2 33.2 mm to (160.0, 60.0)
Connections:
- J1 pad 2: /LMB -> /FWD
- J1 pad 3: /MMB -> /BACK
- J1 pad 4: /RMB -> GND
- R1 pad 2: /LMB -> /FWD
- R2 pad 2: /MMB -> /BACK
- SW1 pad 2: /LMB -> /FWD
- SW2 pad 2: /MMB -> /BACK
Routing:
- net /FWD: track 0.00 -> 34.6 mm, vias 0 -> 2
- net GND: track 0.00 -> 29.3 mm, vias 0 -> 4
- net /BACK: track 0.00 -> 16.7 mm
- net +3V3: track 0.00 -> 14.5 mm, vias 0 -> 2
- added copper zone on B.Cu, net GND
- added copper zone on F.Cu, net GND
Other:
- board outline added: 36 x 12 mm
- board text added: "airMouse-thumb RC1"
