File: hardware/airMouse-thumb/airMouse-thumb.kicad_sch (KiCad schematic)
At the start: 5 parts, among them J2 DS1020-07-4VBT1A-R, SW6 KEY, SW7 KEY

Commit message: thumb pcb
Parts:
- added Logo1: ~, airMouseLib:Bart's Design 30mm, symbol airMouseLib:Bart's_Design_logo
- J1: renamed from J2; footprint (none) -> airMouseLib:DS1020-07-4VBT1A-R
- renumbered R6 to R1, R7 to R2, SW6 to SW1, SW7 to SW2
Other:
- title: EtherPointer -> EtherPointer thumb
Changed lines of the file:
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@@
 	(paper "A4")
 	(title_block
-		(title "EtherPointer")
-		(date "2025-02-13")
+		(title "EtherPointer thumb")
+		(date "2025-02-15")
 		(rev "RC1")
 		(company "Bart's Design")
@@
 		(on_board yes)
 		(dnp no)
-		(property "Reference" "#FLG04"
+		(property "Reference" "#FLG01"
 			(at 151.13 93.345 0)
 			(effects
@@
 			(project "airMouse-mouse"
 				(path "/7db98094-2aea-4dd7-9887-4079cb1655e3"
-					(reference "#FLG04")
+					(reference "#FLG01")
 					(unit 1)
 				)
@@
 		(dnp no)
 		(fields_autoplaced yes)
-		(property "Reference" "#PWR08"
+		(property "Reference" "#PWR01"
 			(at 129.54 93.98 0)
 			(effects
@@
 			(project "airMouse-mouse"
 				(path "/7db98094-2aea-4dd7-9887-4079cb1655e3"
-					(reference "#PWR08")
+					(reference "#PWR01")
 					(unit 1)
 				)
@@
 		(on_board yes)
 		(dnp no)
-		(property "Reference" "R7"
+		(property "Reference" "R2"
 			(at 135.89 90.17 0)
 			(effects
@@
 			(project "airMouse-mouse"
 				(path "/7db98094-2aea-4dd7-9887-4079cb1655e3"
-					(reference "R7")
+					(reference "R2")
+					(unit 1)
+				)
+			)
+		)
+	)
+	(symbol
+		(lib_id "airMouseLib:Bart's_Design_logo")
+		(at 208.28 173.99 0)
+		(unit 1)
+		(exclude_from_sim no)
+		(in_bom yes)
+		(on_board yes)
+		(dnp no)
+		(fields_autoplaced yes)
+		(property "Reference" "Logo1"
+			(at 208.28 170.18 0)
+			(effects
+				(font
+					(size 1.27 1.27)
+				)
+			)
+		)
+		(property "Value" "~"
+			(at 208.28 171.45 0)
+			(effects
+				(font
+					(size 1.27 1.27)
+				)
+			)
+		)
+		(property "Footprint" "airMouseLib:Bart's Design 30mm"
+			(at 208.28 173.99 0)
+			(effects
+				(font
+					(size 1.27 1.27)
+				)
+				(hide yes)
+			)
+		)
+		(property "Datasheet" ""
+			(at 208.28 173.99 0)
+			(effects
+				(font
+					(size 1.27 1.27)
+				)
+				(hide yes)
+			)
+		)
+		(property "Description" ""
+			(at 208.28 173.99 0)
+			(effects
+				(font
+					(size 1.27 1.27)
+				)
+				(hide yes)
+			)
+		)
+		(instances
+			(project ""
+				(path "/7db98094-2aea-4dd7-9887-4079cb1655e3"
+					(reference "Logo1")
 					(unit 1)
 				)
@@
 		(dnp no)
 		(fields_autoplaced yes)
-		(property "Reference" "#PWR09"
+		(property "Reference" "#PWR02"
 			(at 135.89 93.98 0)
 			(effects
@@
 			(project "airMouse-mouse"
 				(path "/7db98094-2aea-4dd7-9887-4079cb1655e3"
-					(reference "#PWR09")
+					(reference "#PWR02")
 					(unit 1)
 				)
@@
 		(dnp no)
 		(fields_autoplaced yes)
-		(property "Reference" "#PWR017"
+		(property "Reference" "#PWR03"
 			(at 143.51 93.98 0)
 			(effects
@@
 			(project "airMouse-mouse"
 				(path "/7db98094-2aea-4dd7-9887-4079cb1655e3"
-					(reference "#PWR017")
+					(reference "#PWR03")
 					(unit 1)
 				)
@@
 		(on_board yes)
 		(dnp no)
-		(property "Reference" "#PWR015"
+		(property "Reference" "#PWR04"
 			(at 95.25 118.11 0)
 			(effects
@@
 			(project "airMouse-mouse"
 				(path "/7db98094-2aea-4dd7-9887-4079cb1655e3"
-					(reference "#PWR015")
+					(reference "#PWR04")
 					(unit 1)
 				)
@@
 		(dnp no)
 		(fields_autoplaced yes)
-		(property "Reference" "#FLG03"
+		(property "Reference" "#FLG02"
 			(at 168.91 109.855 0)
 			(effects
@@
 			(project "airMouse-mouse"
 				(path "/7db98094-2aea-4dd7-9887-4079cb1655e3"
-					(reference "#FLG03")
+					(reference "#FLG02")
 					(unit 1)
 				)
@@
 		(on_board yes)
 		(dnp no)
-		(property "Reference" "SW7"
+		(property "Reference" "SW2"
 			(at 111.76 104.14 0)
 			(effects
@@
 			(project "airMouse-mouse"
 				(path "/7db98094-2aea-4dd7-9887-4079cb1655e3"
-					(reference "SW7")
+					(reference "SW2")
 					(unit 1)
 				)
@@
 		(on_board yes)
 		(dnp no)
-		(property "Reference" "SW6"
+		(property "Reference" "SW1"
 			(at 111.76 100.33 0)
 			(effects
@@
 			(project "airMouse-mouse"
 				(path "/7db98094-2aea-4dd7-9887-4079cb1655e3"
-					(reference "SW6")
+					(reference "SW1")
 					(unit 1)
 				)
@@
 		(dnp no)
 		(fields_autoplaced yes)
-		(property "Reference" "#PWR016"
+		(property "Reference" "#PWR05"
 			(at 156.21 120.65 0)
 			(effects
@@
 			(project "airMouse-mouse"
 				(path "/7db98094-2aea-4dd7-9887-4079cb1655e3"
-					(reference "#PWR016")
+					(reference "#PWR05")
 					(unit 1)
 				)
@@
 		(on_board yes)
 		(dnp no)
-		(property "Reference" "R6"
+		(property "Reference" "R1"
 			(at 129.54 90.17 0)
 			(effects
@@
 			(project "airMouse-mouse"
 				(path "/7db98094-2aea-4dd7-9887-4079cb1655e3"
-					(reference "R6")
+					(reference "R1")
 					(unit 1)
 				)
@@
 		(on_board yes)
 		(dnp no)
-		(property "Reference" "J2"
+		(property "Reference" "J1"
 			(at 158.75 103.2255 0)
 			(effects
@@
 			)
 		)
-		(property "Footprint" ""
+		(property "Footprint" "airMouseLib:DS1020-07-4VBT1A-R"
 			(at 156.21 102.87 0)
 			(effects
@@
 			(project ""
 				(path "/7db98094-2aea-4dd7-9887-4079cb1655e3"
-					(reference "J2")
-					(unit 1)
-				)
+					(reference "J1")
+					(unit 1)
+				)
