File: hardware/airMouse-mcu-proto/airMouse-mcu-proto.kicad_sch (KiCad schematic)
At the start: 58 parts, among them J1 MCU_PRG, J2 RADIO_PRG, J3 AT, Q1 IRLML6346, SW1 KEY, U1 LSM6DS3TR-C, U2 TLV61070ADBV, U3 STM32G071RBTx, U4 ESP32-C3-WROOM-02U

Commit message: working on
Parts:
- removed R55: 0R, symbol Device:R
- R3, R4: footprint (none) -> Resistor_SMD:R_0603_1608Metric
Connections:
- net ESP_3V3 is gone; now on net +3V3: C15.1, C16.1, R12.1, R13.1, R17.1, R18.1, U4.1 (3V3)
- net +3V3: now also C10.1, C11.1, C12.1, C4.1, C5.1, FB1.1, R1.1, R7.1, R8.1, R9.1, U1.5 (VDDIO), U1.8 (VDD), U3.6 (VBAT), U3.8 (VDD); no longer R3.1, R4.1
- net GND: now also R3.2, R4.2; no longer U1.2 (SDX), U1.3 (SCX)
- removed net MCU_3V3: C10.1, C11.1, C12.1, FB1.1, R3.2, R7.1, R8.1, R9.1, U3.6 (VBAT), U3.8 (VDD)
- removed net SENSOR_3V3: C4.1, C5.1, R1.1, R4.2, U1.5 (VDDIO), U1.8 (VDD)
- new net SCX: R4.1, U1.3 (SCX)
- new net SDX: R3.1, U1.2 (SDX)
Other:
- moved on the sheet: C5, R7, R8, R9
