File: hardware/airMouse-mcu/airMouse-mcu.kicad_sch (KiCad schematic)
At the start: 58 parts, among them J1 MCU_PRG, J2 RADIO_PRG, J3 AT, Q1 IRLML6346, SW1 KEY, U1 LSM6DS3TR-C, U2 TLV61070ADBV, U3 STM32G071RBTx, U4 ESP32-C3-WROOM-02U

Commit message: new mcu pcb
Parts:
- removed H1, H2, H3: MountingHole, MountingHole:MountingHole_2.2mm_M2_ISO14580, symbol Mechanical:MountingHole
- removed J3: AT, airMouseLib:JST_ZH_S3B-ZR-SM4A-TF_1x03-1MP_P1.50mm_Horizontal, symbol Connector_Generic_MountingPin:Conn_01x03_MountingPin
- removed U4: ESP32-C3-WROOM-02U, RF_Module:ESP32-C3-WROOM-02U, symbol RF_Module:ESP32-C3-WROOM-02U
- added TP3: AT_MCU_RX, TestPoint:TestPoint_Pad_D1.0mm, symbol Connector:TestPoint
- added TP4: AT_MCU_TX, TestPoint:TestPoint_Pad_D1.0mm, symbol Connector:TestPoint
- added U5: ESP32-C3-WROOM-02, RF_Module:ESP32-C3-WROOM-02, symbol RF_Module:ESP32-C3-WROOM-02
- C7: footprint Capacitor_SMD:C_1206_3216Metric -> Capacitor_SMD:C_0805_2012Metric
- R18: value 10k -> 10k(NM)
- R3, R4, R55: footprint (none) -> Resistor_SMD:R_0603_1608Metric
Connections:
- net AT_MCU_RX: now also TP3.1, U5.6 (IO7)
- net AT_MCU_TX: now also TP4.1, U5.5 (IO6)
- net ESP_3V3: now also U5.1 (3V3)
- net ESP_BOOT: now also U5.8 (IO9)
- net ESP_EN: now also U5.2 (EN)
- net GND: now also U5.19 (GND), U5.9 (GND)
- net PRG_ESP_RX: now also U5.11 (IO20/RXD)
- net PRG_ESP_TX: now also U5.12 (IO21/TXD)
- net at R17.2: now also U5.16 (IO2)
- net at R13.2: now also U5.7 (IO8)
Other:
- note added: "DONE much much wider BAT- width DEPRECATED step up voltage from BAT(charge pump) DEPRECATED Add acc circuit DEPRECATED Add power switches for peripherals(ESP32, gyro sensor) make place for ESP32 with pcb antenna EN have to be push pull, other wise voltage on this pin can't rise. why? place buffer capacitor on battery"
- note removed: "remove R3/R4 C7- change to 0805 change converter to: TLV61070A much much wider BAT- width step up voltage from BAT(charge pump) Add acc circuit Add power switches for peripherals(ESP32, gyro sensor) make place for ESP32 with pcb antenna EN have to be push pull, other wise voltage on this pin can't rise. why? place buffer capacitor on battery"

Commit message: new mcu-pcb
Other:
- title: EtherPointer mcu -> Neuro Glider
Changed lines of the file:
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@@
 	(paper "A4")
 	(title_block
-		(title "EtherPointer mcu")
-		(date "2025-02-15")
-		(rev "RC1")
+		(title "Neuro Glider")
+		(date "2025-03-21")
+		(rev "v1.0")
 		(company "Bart's Design")
 		(comment 1 "Bartosz Pracz")
@@
 	)
 	(junction
+		(at 72.39 148.59)
+		(diameter 0)
+		(color 0 0 0 0)
+	)
+	(junction
 		(at 101.6 22.86)
 		(diameter 0)
@@
 	)
 	(junction
+		(at 270.51 101.6)
+		(diameter 0)
+		(color 0 0 0 0)
+	)
+	(junction
 		(at 34.29 170.18)
 		(diameter 0)
@@
 	)
 	(junction
+		(at 162.56 36.83)
+		(diameter 0)
+		(color 0 0 0 0)
+	)
+	(junction
 		(at 142.24 41.91)
 		(diameter 0)
@@
 	(wire
 		(pts
+			(xy 72.39 144.78) (xy 72.39 148.59)
+		)
+		(stroke
+			(width 0)
+			(type default)
+		)
+	)
+	(wire
+		(pts
 			(xy 162.56 125.73) (xy 171.45 125.73)
 		)
@@
 	(wire
 		(pts
+			(xy 162.56 33.02) (xy 162.56 36.83)
+		)
+		(stroke
+			(width 0)
+			(type default)
+		)
+	)
+	(wire
+		(pts
 			(xy 59.69 148.59) (xy 59.69 157.48)
 		)
@@
 	)
 	(symbol
+		(lib_id "power:PWR_FLAG")
+		(at 72.39 144.78 0)
+		(unit 1)
+		(exclude_from_sim no)
+		(in_bom yes)
+		(on_board yes)
+		(dnp no)
+		(fields_autoplaced yes)
+		(property "Reference" "#FLG04"
+			(at 72.39 142.875 0)
+			(effects
+				(font
+					(size 1.27 1.27)
+				)
+				(hide yes)
+			)
+		)
+		(property "Value" "PWR_FLAG"
+			(at 72.39 139.7 0)
+			(effects
+				(font
+					(size 1.27 1.27)
+				)
+			)
+		)
+		(property "Footprint" ""
+			(at 72.39 144.78 0)
+			(effects
+				(font
+					(size 1.27 1.27)
+				)
+				(hide yes)
+			)
+		)
+		(property "Datasheet" "~"
+			(at 72.39 144.78 0)
+			(effects
+				(font
+					(size 1.27 1.27)
+				)
+				(hide yes)
+			)
+		)
+		(property "Description" "Special symbol for telling ERC where power comes from"
+			(at 72.39 144.78 0)
+			(effects
+				(font
+					(size 1.27 1.27)
+				)
+				(hide yes)
+			)
+		)
+		(pin "1"
+		)
+		(instances
+			(project "airMouse-mcu"
+				(path "/7db98094-2aea-4dd7-9887-4079cb1655e3"
+					(reference "#FLG04")
+					(unit 1)
+				)
+			)
+		)
+	)
+	(symbol
 		(lib_id "power:GND")
 		(at 162.56 44.45 0)
@@
 	)
 	(symbol
+		(lib_id "power:PWR_FLAG")
+		(at 162.56 33.02 0)
+		(unit 1)
+		(exclude_from_sim no)
+		(in_bom yes)
+		(on_board yes)
+		(dnp no)
+		(fields_autoplaced yes)
+		(property "Reference" "#FLG05"
+			(at 162.56 31.115 0)
+			(effects
+				(font
+					(size 1.27 1.27)
+				)
+				(hide yes)
+			)
+		)
+		(property "Value" "PWR_FLAG"
+			(at 162.56 27.94 0)
+			(effects
+				(font
+					(size 1.27 1.27)
+				)
+			)
+		)
+		(property "Footprint" ""
+			(at 162.56 33.02 0)
+			(effects
+				(font
+					(size 1.27 1.27)
+				)
+				(hide yes)
+			)
+		)
+		(property "Datasheet" "~"
+			(at 162.56 33.02 0)
+			(effects
+				(font
+					(size 1.27 1.27)
+				)
+				(hide yes)
+			)
+		)
+		(property "Description" "Special symbol for telling ERC where power comes from"
+			(at 162.56 33.02 0)
+			(effects
+				(font
+					(size 1.27 1.27)
+				)
+				(hide yes)
+			)
+		)
+		(pin "1"
+		)
+		(instances
+			(project "airMouse-mcu"
+				(path "/7db98094-2aea-4dd7-9887-4079cb1655e3"
+					(reference "#FLG05")
+					(unit 1)
+				)
+			)
+		)
+	)
+	(symbol
 		(lib_id "Device:C")
 		(at 43.18 27.94 0)
@@
 					(unit 1)
 				)
+			)
+		)
+	)
+	(symbol
+		(lib_id "power:PWR_FLAG")
+		(at 270.51 101.6 0)
+		(unit 1)
+		(exclude_from_sim no)
+		(in_bom yes)
+		(on_board yes)
+		(dnp no)
+		(fields_autoplaced yes)
+		(property "Reference" "#FLG03"
+			(at 270.51 99.695 0)
+			(effects
+				(font
+					(size 1.27 1.27)
+				)
+				(hide yes)
+			)
+		)
+		(property "Value" "PWR_FLAG"
+			(at 270.51 96.52 0)
+			(effects
+				(font
+					(size 1.27 1.27)
+				)
+			)
+		)
+		(property "Footprint" ""
+			(at 270.51 101.6 0)
+			(effects
+				(font
+					(size 1.27 1.27)
+				)
+				(hide yes)
+			)
+		)
+		(property "Datasheet" "~"
+			(at 270.51 101.6 0)
+			(effects
+				(font
+					(size 1.27 1.27)
+				)
+				(hide yes)
+			)
+		)
+		(property "Description" "Special symbol for telling ERC where power comes from"
+			(at 270.51 101.6 0)
+			(effects
+				(font
+					(size 1.27 1.27)
+				)
+				(hide yes)
+			)
+		)
+		(pin "1"
+		)
+		(instances
+			(project ""
+				(path "/7db98094-2aea-4dd7-9887-4079cb1655e3"
+					(reference "#FLG03")
+					(unit 1)
+				)
